File: Chapter06/src/oscilloscope-circuit/ADC.sch (KiCad schematic (older format))
At the start: 30 parts, among them U1 LTC2267-14

Commit message: Working on chapter 6
Parts:
- U1: symbol Oscilloscope:LTC2267-14 -> Schematic_Symbols:LTC2267-14
Changed lines of the file:
@@
 	7950 2950 7950 2350
 $Comp
-L Oscilloscope:LTC2267-14 U1
+L Schematic_Symbols:LTC2267-14 U1
 U 1 1 5F68C778
 P 5350 3550
