File: Chapter06/src/oscilloscope-circuit/Analog Inputs.sch (KiCad schematic (older format))
At the start: 24 parts, among them J1 Ch1 BNC, U6 GDT CG775, U7 ADA4817-1, U8 LT6411

Commit message: Working on chapter 6
Parts:
- U6: footprint Oscilloscope_footprints:Littelfuse-GTCC23-XXXM-R01-2-Series-GDT -> Footprints:Littelfuse-GTCC23-XXXM-R01-2-Series-GDT; symbol Oscilloscope:GDT -> Schematic_Symbols:GDT
- U7: symbol Oscilloscope:ADA4817-1 -> Schematic_Symbols:ADA4817-1
- U8: symbol Oscilloscope:LT6411 -> Schematic_Symbols:LT6411
Changed lines of the file:
@@
 	5600 4350 5600 4900
 $Comp
-L Oscilloscope:+3V0 #PWR047
+L Schematic_Symbols:+3V0 #PWR047
 U 1 1 5F70574E
 P 5600 3050
@@
 	5600 3750 5600 3150
 $Comp
-L Oscilloscope:GDT U6
+L Schematic_Symbols:GDT U6
 U 1 1 5F70AA56
 P 2300 3800
 F 0 "U6" V 2254 3978 50  0000 L CNN
 F 1 "GDT CG775" V 2345 3978 50  0000 L CNN
-F 2 "Oscilloscope_footprints:Littelfuse-GTCC23-XXXM-R01-2-Series-GDT" H 2300 3800 50  0001 C CNN
+F 2 "Footprints:Littelfuse-GTCC23-XXXM-R01-2-Series-GDT" H 2300 3800 50  0001 C CNN
 F 3 "" H 2300 3800 50  0001 C CNN
 	1    2300 3800
@@
 	5600 4900 6200 4900
 $Comp
-L Oscilloscope:-3V0 #PWR048
+L Schematic_Symbols:-3V0 #PWR048
 U 1 1 5F73C0E6
 P 5600 4950
@@
 Input range ±10 V\nwith 1X probe
 $Comp
-L Oscilloscope:LT6411 U8
+L Schematic_Symbols:LT6411 U8
 U 1 1 5F76C21F
 P 8500 4250
@@
 $EndComp
 $Comp
-L Oscilloscope:-3V0 #PWR058
+L Schematic_Symbols:-3V0 #PWR058
 U 1 1 5F7800EE
 P 8550 5300
@@
 Connection ~ 9900 3050
 $Comp
-L Oscilloscope:+3V0 #PWR057
+L Schematic_Symbols:+3V0 #PWR057
 U 1 1 5F95149A
 P 8500 2950
@@
 	9150 4500 10250 4500
 $Comp
-L Oscilloscope:-3V0 #PWR062
+L Schematic_Symbols:-3V0 #PWR062
 U 1 1 5F506043
 P 10400 3500
@@
 $EndComp
 $Comp
-L Oscilloscope:ADA4817-1 U7
+L Schematic_Symbols:ADA4817-1 U7
 U 1 1 5F743611
 P 5700 4050
@@
 	5800 4350 5800 4400
 $Comp
-L Oscilloscope:+3V0 #PWR050
+L Schematic_Symbols:+3V0 #PWR050
 U 1 1 5F7578C6
 P 6050 4400
