File: Chapter06/src/oscilloscope-circuit/Calibration.sch (KiCad schematic (older format))
At the start: 12 parts, among them J5 1 KHz ±3.0V, J6 GND, J7 3.0VDC, J8 -3.0VDC, U9 TLV2371DBV

Commit message: Working on chapter 6
Changed lines of the file:
@@
 $EndComp
 $Comp
-L Oscilloscope:+3V0 #PWR076
+L Schematic_Symbols:+3V0 #PWR076
 U 1 1 5F9CBDEC
 P 7950 2450
@@
 $EndComp
 $Comp
-L Oscilloscope:-3V0 #PWR077
+L Schematic_Symbols:-3V0 #PWR077
 U 1 1 5F9D0C59
 P 8700 3550
@@
 $EndComp
 $Comp
-L +1v8:+1V8 #PWR071
+L power:+1V8 #PWR071
 U 1 1 5F9FFEE7
 P 3500 3250
@@
 $EndComp
 $Comp
-L Oscilloscope:+3V0 #PWR073
+L Schematic_Symbols:+3V0 #PWR073
 U 1 1 5F741EEB
 P 4400 2550
@@
 $EndComp
 $Comp
-L Oscilloscope:-3V0 #PWR074
+L Schematic_Symbols:-3V0 #PWR074
 U 1 1 5F742716
 P 4400 3550
