File: Chapter06/src/oscilloscope-circuit/Oscilloscope.kicad_pcb (KiCad board)
At the start: 4 copper layers, 63.5 x 63.5 mm, 84 parts, among them J1 Ch1 BNC, J2 PMOD B, J3 PMOD C, J4 SPI header, J5 1 KHz ±3.0V, J6 GND, J7 3.0VDC, J8 -3.0VDC, U1 LTC2267-14, U2 TLV75718PDBV, U3 MIC5501-3.0YM5, U4 LM2776, U5 TC59, U6 GDT CG775, U7 ADA4817-1, U8 LT6411, U9 TLV2371DBV

Commit message: Working on chapter 6
Parts:
- J2, J3: footprint Oscilloscope footprints:PinHeader_2x06_P2.54mm_renumbered -> Footprints:PinHeader_2x06_P2.54mm_renumbered
- U6: footprint Oscilloscope_footprints:Littelfuse-GTCC23-XXXM-R01-2-Series-GDT -> Footprints:Littelfuse-GTCC23-XXXM-R01-2-Series-GDT
