File: Chapter06/src/oscilloscope-circuit/PMOD Ports.sch (KiCad schematic (older format))
At the start: 2 parts, among them J2 PMOD B, J3 PMOD C

Commit message: Working on chapter 6
Parts:
- J2, J3: footprint Oscilloscope footprints:PinHeader_2x06_P2.54mm_renumbered -> Footprints:PinHeader_2x06_P2.54mm_renumbered
Changed lines of the file:
@@
 F 0 "J2" H 3650 3267 50  0000 C CNN
 F 1 "PMOD B" H 3650 3176 50  0000 C CNN
-F 2 "Oscilloscope footprints:PinHeader_2x06_P2.54mm_renumbered" H 3600 2850 50  0001 C CNN
+F 2 "Footprints:PinHeader_2x06_P2.54mm_renumbered" H 3600 2850 50  0001 C CNN
 F 3 "~" H 3600 2850 50  0001 C CNN
 	1    3600 2850
@@
 F 0 "J3" H 7200 3317 50  0000 C CNN
 F 1 "PMOD C" H 7200 3226 50  0000 C CNN
-F 2 "Oscilloscope footprints:PinHeader_2x06_P2.54mm_renumbered" H 7150 2900 50  0001 C CNN
+F 2 "Footprints:PinHeader_2x06_P2.54mm_renumbered" H 7150 2900 50  0001 C CNN
 F 3 "~" H 7150 2900 50  0001 C CNN
 	1    7150 2900
